Commit message: obstacle avoidance

File: catkin_ws/src/bot_base/urdf/bot.urdf (robot description, URDF)
Before this commit: robot bot, 3 links, 2 joints
Links:
- removed link camera
Joints:
- removed joint camera
- joint zed_mini: origin xyz=0 0 0 rpy=-1.57 0 -1.57 -> xyz=0.075 0.025 0.15 rpy=0 0.3488888888888889 0; parent camera -> base_link

Commit message: kernal func pass by value

File: catkin_ws/src/bot_base/urdf/bot.urdf (robot description, URDF)
Before this commit: robot bot, 2 links, 1 joints
Joints:
- joint zed_mini: origin xyz=0.075 0.025 0.15 rpy=0 0.3488888888888889 0 -> xyz=0 0 0 rpy=0 0.3488888888888889 0
